File: hw/sch_pcb/PCRD08.kicad_pcb (KiCad board)
At the start: 2 copper layers, 70.6 x 40.1 mm, 65 parts, among them J201 MCX, J202 HEADER_2x01, J301 HEADER_2x03, J302 HEADER_2x08, M103 HOLE, M201 RFShield_TwoPieces, U201 AD8691, U202 ISL21080DIH309, U203 TS3021ILT, U204 AD8691, U205 SN74LVC2G74, U206 ISL21080CIH341Z-TK, U207 LTC1865-MS, U301 TXU0304PWR, U302 SN74LVC1G125DCKT, U303 MIC5504-3.3YM5-TR

Commit message: Rename project PCRD008 -> PCRD08 to match MLAB module naming convention
Other:
- board text added: "PCRD08"
- board text removed: "PCRD008"
Changed lines of the file:
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@@
 	(paper "A4")
 	(title_block
-		(title "PCRD008")
+		(title "PCRD08")
 		(date "2026-07-24")
 		(company "Universal Scientific Technologies s.r.o.")
@@
 		)
 	)
-	(gr_text "PCRD008"
+	(gr_text "PCRD08"
 		(at 133.4 129.1 0)
 		(layer "F.SilkS")
