File: hw/sch_pcb/analogue_backend.kicad_sch (KiCad schematic)
At the start: 47 parts, among them J201 MCX, J202 HEADER_2x01, M201 RFShield_TwoPieces, U201 AD8691, U202 ISL21080DIH309, U203 TS3021ILT, U204 AD8691, U205 SN74LVC2G74, U206 ISL21080CIH341Z-TK, U207 LTC1865-MS

Commit message: Rename project PCRD008 -> PCRD08 to match MLAB module naming convention
Other:
- title: PCRD008 -> PCRD08
Changed lines of the file:
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@@
 	(paper "A4")
 	(title_block
-		(title "PCRD008")
+		(title "PCRD08")
 		(date "2026-7-24")
 		(company "KubFire <info@ust.cz>")

Commit message: Remove resolved TODO notes on R206/R207/R208/C213 gain check
Verified U201 AC-coupled non-inverting stage: signal path enters the
+ input via C211, so it cannot invert, and the R206/R207/R208/C213
network algebraically settles to unity gain at high frequency
regardless of exact values (confirmed numerically with the populated
values: phase stays within ±90°, |H|→1 above ~10 MHz).
Other:
- note removed: "pls zkontrolovat ze R208, R207, R206 a C213 maji spravne hodnoty aby to neinvertovalo a melo 1x gain pro vysoke frekvence, dekuji"
Changed lines of the file:
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@@
-		)
-	)
-	(text "pls zkontrolovat ze R208, R207, R206 a C213\nmaji spravne hodnoty aby to neinvertovalo a \nmelo 1x gain pro vysoke frekvence, dekuji "
-		(exclude_from_sim no)
-		(at 70.104 145.288 0)
-		(effects
-			(font
-				(size 1.524 1.524)
-			)
 		)
 	)

Commit message: Re-anotate schematics.
Parts:
- renumbered C201 to C1, C210 to C10, C211 to C11, C212 to C12, C213 to C13, C214 to C14, C215 to C15, C216 to C16, C217 to C17, C218 to C18, C219 to C19, C202 to C2, C220 to C20, C221 to C21, C203 to C3, C204 to C4, C205 to C5, C206 to C6, C207 to C7, C208 to C8, C209 to C9, J201 to J1, J202 to J2, JP201 to JP1, L201 to L1, M201 to M5, R201 to R1, R210 to R10, R211 to R11, R202 to R2, R203 to R3, R204 to R4, R205 to R5, R206 to R6, R207 to R7, R208 to R8, R209 to R9, TP201 to TP1, TP202 to TP2, TP203 to TP3, U201 to U1, U202 to U2, U203 to U3, U204 to U4, U205 to U5, U206 to U6, U207 to U7
