File: hw/sch_pcb/interface.kicad_sch (KiCad schematic)
At the start: 16 parts, among them J301 HEADER_2x03, J302 HEADER_2x08, U301 TXU0304PWR, U302 SN74LVC1G125DCKT, U303 MIC5504-3.3YM5-TR

Commit message: Rename project PCRD008 -> PCRD08 to match MLAB module naming convention
Other:
- title: PCRD008 -> PCRD08
Changed lines of the file:
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@@
 	(paper "A4")
 	(title_block
-		(title "PCRD008")
+		(title "PCRD08")
 		(date "2026-07-24")
 		(company "KubFire <info@ust.cz>")

Commit message: Update submodule and workflow.
Parts:
- U301: DESCRIPTION Translation - Voltage Levels Four channel unidirectional le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 -> (none)

Commit message: Re-anotate schematics.
Parts:
- renumbered C301 to C22, C302 to C23, C303 to C24, C304 to C25, C305 to C26, C307 to C27, C306 to C28, C308 to C29, C309 to C30, C310 to C31, J302 to J3, J301 to J4, L301 to L2, U303 to U10, U301 to U8, U302 to U9
